File: RFModulator1.kicad_pcb (KiCad board)
At the start: 2 copper layers, 50 x 64 mm, 19 parts, among them J1 Conn_Coaxial, J2 Conn_Coaxial, J3 Conn_Coaxial, P1 10K, P2 10K, Q2 Q_NJFET_GDS

Commit message: with jst
Parts:
- removed +15V, GND: +15VHole, Library:Pin Through Hole
- added J4: Conn_01x02_Socket, Connector_JST:JST_XH_B2B-XH-A_1x02_P2.50mm_Vertical, F.Cu at (179.5, 105.5)
Other:
- board size 50 x 64 mm -> 50 x 66.9 mm
